File: hardware/circuit_board/_autosave-sound_laser.kicad_sch (KiCad schematic)
At the start: 51 parts, among them J1 Conn_01x02, J2 Conn_01x02, J3 Conn_01x02, J4 Conn_01x02, J5 Conn_01x02, J6 Conn_01x02, J7 Conn_01x02, M1 Ultrasonic_Transducer, M10 Ultrasonic_Transducer, M11 Ultrasonic_Transducer, M12 Ultrasonic_Transducer, M13 Ultrasonic_Transducer, M14 Ultrasonic_Transducer, M15 Ultrasonic_Transducer, M16 Ultrasonic_Transducer, M17 Ultrasonic_Transducer, M18 Ultrasonic_Transducer, M19 Ultrasonic_Transducer, M2 Ultrasonic_Transducer, M3 Ultrasonic_Transducer, M4 Ultrasonic_Transducer, M5 Ultrasonic_Transducer, M6 Ultrasonic_Transducer, M7 Ultrasonic_Transducer, M8 Ultrasonic_Transducer, M9 Ultrasonic_Transducer, U1 LTC2631-Z, U2 LM2735XMF

Commit message: ADD i2c Resistor calculation, REWORK power supplay
Parts:
- J1, J2, J3, J4, J5, J6: value Conn_01x02 -> JST SH BM02B Connector
Changed lines of the file:
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@@
     (in_bom yes) (on_board yes) (fields_autoplaced)
     (property "Reference" "J3" (id 0) (at 191.77 120.65 0))
-    (property "Value" "Conn_01x02" (id 1) (at 191.77 120.65 0)
+    (property "Value" "JST SH BM02B Connector" (id 1) (at 191.77 120.65 0)
       (effects (font (size 1.27 1.27)) hide)
     )
@@
     (in_bom yes) (on_board yes) (fields_autoplaced)
     (property "Reference" "J2" (id 0) (at 200.66 120.65 0))
-    (property "Value" "Conn_01x02" (id 1) (at 200.66 120.65 0)
+    (property "Value" "JST SH BM02B Connector" (id 1) (at 200.66 120.65 0)
       (effects (font (size 1.27 1.27)) hide)
     )
@@
     (in_bom yes) (on_board yes) (fields_autoplaced)
     (property "Reference" "J5" (id 0) (at 173.99 120.65 0))
-    (property "Value" "Conn_01x02" (id 1) (at 173.99 120.65 0)
+    (property "Value" "JST SH BM02B Connector" (id 1) (at 173.99 120.65 0)
       (effects (font (size 1.27 1.27)) hide)
     )
@@
     (in_bom yes) (on_board yes) (fields_autoplaced)
     (property "Reference" "J1" (id 0) (at 209.55 120.65 0))
-    (property "Value" "Conn_01x02" (id 1) (at 209.55 120.65 0)
+    (property "Value" "JST SH BM02B Connector" (id 1) (at 209.55 120.65 0)
       (effects (font (size 1.27 1.27)) hide)
     )
@@
     (in_bom yes) (on_board yes) (fields_autoplaced)
     (property "Reference" "J6" (id 0) (at 165.1 120.65 0))
-    (property "Value" "Conn_01x02" (id 1) (at 165.1 120.65 0)
+    (property "Value" "JST SH BM02B Connector" (id 1) (at 165.1 120.65 0)
       (effects (font (size 1.27 1.27)) hide)
     )
@@
     (in_bom yes) (on_board yes) (fields_autoplaced)
     (property "Reference" "J4" (id 0) (at 182.88 120.65 0))
-    (property "Value" "Conn_01x02" (id 1) (at 182.88 120.65 0)
+    (property "Value" "JST SH BM02B Connector" (id 1) (at 182.88 120.65 0)
       (effects (font (size 1.27 1.27)) hide)
     )
@@
     )
     (path "/b893555e-743d-4cf9-bd5a-f020e2718f96"
-      (reference "J1") (unit 1) (value "Conn_01x02") (footprint "Connector_JST:JST_SH_BM02B-SRSS-TB_1x02-1MP_P1.00mm_Vertical")
+      (reference "J1") (unit 1) (value "JST SH BM02B Connector") (footprint "Connector_JST:JST_SH_BM02B-SRSS-TB_1x02-1MP_P1.00mm_Vertical")
     )
     (path "/41f187f0-c6dd-43c8-8895-eac8ebc41199"
-      (reference "J2") (unit 1) (value "Conn_01x02") (footprint "Connector_JST:JST_SH_BM02B-SRSS-TB_1x02-1MP_P1.00mm_Vertical")
+      (reference "J2") (unit 1) (value "JST SH BM02B Connector") (footprint "Connector_JST:JST_SH_BM02B-SRSS-TB_1x02-1MP_P1.00mm_Vertical")
     )
     (path "/1b3a272c-48df-47fd-b37c-cee5898d6c9a"
-      (reference "J3") (unit 1) (value "Conn_01x02") (footprint "Connector_JST:JST_SH_BM02B-SRSS-TB_1x02-1MP_P1.00mm_Vertical")
+      (reference "J3") (unit 1) (value "JST SH BM02B Connector") (footprint "Connector_JST:JST_SH_BM02B-SRSS-TB_1x02-1MP_P1.00mm_Vertical")
     )
     (path "/f454f6b8-6542-4029-aa53-85ac46fe0b4b"
-      (reference "J4") (unit 1) (value "Conn_01x02") (footprint "Connector_JST:JST_SH_BM02B-SRSS-TB_1x02-1MP_P1.00mm_Vertical")
+      (reference "J4") (unit 1) (value "JST SH BM02B Connector") (footprint "Connector_JST:JST_SH_BM02B-SRSS-TB_1x02-1MP_P1.00mm_Vertical")
     )
     (path "/9b7695b7-9db0-4c8e-9077-f8b7d4d3a13e"
-      (reference "J5") (unit 1) (value "Conn_01x02") (footprint "Connector_JST:JST_SH_BM02B-SRSS-TB_1x02-1MP_P1.00mm_Vertical")
+      (reference "J5") (unit 1) (value "JST SH BM02B Connector") (footprint "Connector_JST:JST_SH_BM02B-SRSS-TB_1x02-1MP_P1.00mm_Vertical")
     )
     (path "/cb8e411a-1cc5-4c53-9eeb-4024c1c299a0"
-      (reference "J6") (unit 1) (value "Conn_01x02") (footprint "Connector_JST:JST_SH_BM02B-SRSS-TB_1x02-1MP_P1.00mm_Vertical")
+      (reference "J6") (unit 1) (value "JST SH BM02B Connector") (footprint "Connector_JST:JST_SH_BM02B-SRSS-TB_1x02-1MP_P1.00mm_Vertical")
     )
     (path "/6746b76e-fcdf-48a8-9cd1-db639066bc4d"
