File: hardware/circuit_board/sound_laser.kicad_sch (KiCad schematic)
At the start: 51 parts, among them J1 Conn_01x02, J2 Conn_01x02, J3 Conn_01x02, J4 Conn_01x02, J5 Conn_01x02, J6 Conn_01x02, J7 Conn_01x02, M1 Ultrasonic_Transducer, M10 Ultrasonic_Transducer, M11 Ultrasonic_Transducer, M12 Ultrasonic_Transducer, M13 Ultrasonic_Transducer, M14 Ultrasonic_Transducer, M15 Ultrasonic_Transducer, M16 Ultrasonic_Transducer, M17 Ultrasonic_Transducer, M18 Ultrasonic_Transducer, M19 Ultrasonic_Transducer, M2 Ultrasonic_Transducer, M3 Ultrasonic_Transducer, M4 Ultrasonic_Transducer, M5 Ultrasonic_Transducer, M6 Ultrasonic_Transducer, M7 Ultrasonic_Transducer, M8 Ultrasonic_Transducer, M9 Ultrasonic_Transducer, U1 LTC2631-Z, U2 LM2735XMF

Commit message: REWORK circuit board
Parts:
- J1, J2, J3, J4, J5, J6: value Conn_01x02 -> JST SH BM02B Connector
- J7: footprint Connector_JST:JST_PH_B2B-PH-SM4-TB_1x02-1MP_P2.00mm_Vertical -> Connector_JST:JST_PH_B2B-PH-K_1x02_P2.00mm_Vertical
- R5, R6: value R -> 1.7k
Other:
- moved on the sheet: R6
Changed lines of the file:
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@@
   (junction (at 128.27 149.86) (diameter 0) (color 0 0 0 0)
   )
+  (junction (at 248.92 127) (diameter 0) (color 0 0 0 0)
+  )
   (junction (at 121.92 168.91) (diameter 0) (color 0 0 0 0)
   )
@@
   (junction (at 179.07 127) (diameter 0) (color 0 0 0 0)
   )
-  (junction (at 247.65 127) (diameter 0) (color 0 0 0 0)
-  )
   (junction (at 60.96 149.86) (diameter 0) (color 0 0 0 0)
   )
@@
     (stroke (width 0) (type default) (color 0 0 0 0))
   )
-  (wire (pts (xy 247.65 114.3) (xy 247.65 115.57))
+  (wire (pts (xy 248.92 114.3) (xy 248.92 115.57))
     (stroke (width 0) (type default) (color 0 0 0 0))
   )
@@
     (stroke (width 0) (type default) (color 0 0 0 0))
   )
+  (wire (pts (xy 248.92 127) (xy 266.7 127))
+    (stroke (width 0) (type default) (color 0 0 0 0))
+  )
   (wire (pts (xy 212.09 72.39) (xy 212.09 74.93))
     (stroke (width 0) (type default) (color 0 0 0 0))
@@
     (stroke (width 0) (type default) (color 0 0 0 0))
   )
-  (wire (pts (xy 247.65 123.19) (xy 247.65 127))
+  (wire (pts (xy 248.92 123.19) (xy 248.92 127))
     (stroke (width 0) (type default) (color 0 0 0 0))
   )
@@
     (stroke (width 0) (type default) (color 0 0 0 0))
   )
-  (wire (pts (xy 247.65 127) (xy 266.7 127))
-    (stroke (width 0) (type default) (color 0 0 0 0))
-  )
   (wire (pts (xy 90.17 160.02) (xy 83.82 160.02))
     (stroke (width 0) (type default) (color 0 0 0 0))
@@
     (stroke (width 0) (type default) (color 0 0 0 0))
   )
-  (wire (pts (xy 214.63 127) (xy 247.65 127))
+  (wire (pts (xy 214.63 127) (xy 248.92 127))
     (stroke (width 0) (type default) (color 0 0 0 0))
   )
@@
     (in_bom yes) (on_board yes) (fields_autoplaced)
     (property "Reference" "J3" (id 0) (at 191.77 120.65 0))
-    (property "Value" "Conn_01x02" (id 1) (at 191.77 120.65 0)
+    (property "Value" "JST SH BM02B Connector" (id 1) (at 191.77 120.65 0)
       (effects (font (size 1.27 1.27)) hide)
     )
@@
     (pin "2")
   )
-  (symbol (lib_id "Device:R") (at 247.65 119.38 0) (unit 1)
-    (in_bom yes) (on_board yes)
-    (property "Reference" "R6" (id 0) (at 248.92 119.38 0)
-      (effects (font (size 1.27 1.27)) (justify left))
-    )
-    (property "Value" "R" (id 1) (at 248.92 120.65 0)
-      (effects (font (size 1.27 1.27)) (justify left) hide)
-    )
-    (property "Footprint" "Resistor_SMD:R_0805_2012Metric" (id 2) (at 245.872 119.38 90)
-      (effects (font (size 1.27 1.27)) hide)
-    )
-    (property "Datasheet" "~" (id 3) (at 247.65 119.38 0)
+  (symbol (lib_id "Device:R") (at 248.92 119.38 0) (unit 1)
+    (in_bom yes) (on_board yes)
+    (property "Reference" "R6" (id 0) (at 250.19 118.11 0)
+      (effects (font (size 1.27 1.27)) (justify left))
+    )
+    (property "Value" "1.7k" (id 1) (at 250.19 120.65 0)
+      (effects (font (size 1.27 1.27)) (justify left))
+    )
+    (property "Footprint" "Resistor_SMD:R_0805_2012Metric" (id 2) (at 247.142 119.38 90)
+      (effects (font (size 1.27 1.27)) hide)
+    )
+    (property "Datasheet" "~" (id 3) (at 248.92 119.38 0)
       (effects (font (size 1.27 1.27)) hide)
     )
@@
     (in_bom yes) (on_board yes) (fields_autoplaced)
     (property "Reference" "J2" (id 0) (at 200.66 120.65 0))
-    (property "Value" "Conn_01x02" (id 1) (at 200.66 120.65 0)
+    (property "Value" "JST SH BM02B Connector" (id 1) (at 200.66 120.65 0)
       (effects (font (size 1.27 1.27)) hide)
     )
@@
       (effects (font (size 1.27 1.27)) hide)
     )
-    (property "Footprint" "Connector_JST:JST_PH_B2B-PH-SM4-TB_1x02-1MP_P2.00mm_Vertical" (id 2) (at 165.1 110.49 0)
+    (property "Footprint" "Connector_JST:JST_PH_B2B-PH-K_1x02_P2.00mm_Vertical" (id 2) (at 165.1 110.49 0)
       (effects (font (size 1.27 1.27)) hide)
     )
@@
   (symbol (lib_id "Device:R") (at 241.3 119.38 0) (unit 1)
     (in_bom yes) (on_board yes)
-    (property "Reference" "R5" (id 0) (at 242.57 119.38 0)
-      (effects (font (size 1.27 1.27)) (justify left))
-    )
-    (property "Value" "R" (id 1) (at 242.57 120.65 0)
-      (effects (font (size 1.27 1.27)) (justify left) hide)
+    (property "Reference" "R5" (id 0) (at 242.57 118.11 0)
+      (effects (font (size 1.27 1.27)) (justify left))
+    )
+    (property "Value" "1.7k" (id 1) (at 242.57 120.65 0)
+      (effects (font (size 1.27 1.27)) (justify left))
     )
     (property "Footprint" "Resistor_SMD:R_0805_2012Metric" (id 2) (at 239.522 119.38 90)
@@
     (in_bom yes) (on_board yes) (fields_autoplaced)
     (property "Reference" "J5" (id 0) (at 173.99 120.65 0))
-    (property "Value" "Conn_01x02" (id 1) (at 173.99 120.65 0)
+    (property "Value" "JST SH BM02B Connector" (id 1) (at 173.99 120.65 0)
       (effects (font (size 1.27 1.27)) hide)
     )
@@
     (in_bom yes) (on_board yes) (fields_autoplaced)
     (property "Reference" "J1" (id 0) (at 209.55 120.65 0))
-    (property "Value" "Conn_01x02" (id 1) (at 209.55 120.65 0)
+    (property "Value" "JST SH BM02B Connector" (id 1) (at 209.55 120.65 0)
       (effects (font (size 1.27 1.27)) hide)
     )
@@
     (pin "1")
   )
-  (symbol (lib_id "power:+5V") (at 247.65 114.3 0) (unit 1)
-    (in_bom yes) (on_board yes) (fields_autoplaced)
-    (property "Reference" "#PWR0116" (id 0) (at 247.65 118.11 0)
-      (effects (font (size 1.27 1.27)) hide)
-    )
-    (property "Value" "+5V" (id 1) (at 247.65 109.22 0))
-    (property "Footprint" "" (id 2) (at 247.65 114.3 0)
-      (effects (font (size 1.27 1.27)) hide)
-    )
-    (property "Datasheet" "" (id 3) (at 247.65 114.3 0)
+  (symbol (lib_id "power:+5V") (at 248.92 114.3 0) (unit 1)
+    (in_bom yes) (on_board yes) (fields_autoplaced)
+    (property "Reference" "#PWR0116" (id 0) (at 248.92 118.11 0)
+      (effects (font (size 1.27 1.27)) hide)
+    )
+    (property "Value" "+5V" (id 1) (at 248.92 109.22 0))
+    (property "Footprint" "" (id 2) (at 248.92 114.3 0)
+      (effects (font (size 1.27 1.27)) hide)
+    )
+    (property "Datasheet" "" (id 3) (at 248.92 114.3 0)
       (effects (font (size 1.27 1.27)) hide)
     )
@@
     (in_bom yes) (on_board yes) (fields_autoplaced)
     (property "Reference" "J6" (id 0) (at 165.1 120.65 0))
-    (property "Value" "Conn_01x02" (id 1) (at 165.1 120.65 0)
+    (property "Value" "JST SH BM02B Connector" (id 1) (at 165.1 120.65 0)
       (effects (font (size 1.27 1.27)) hide)
     )
@@
     (in_bom yes) (on_board yes) (fields_autoplaced)
     (property "Reference" "J4" (id 0) (at 182.88 120.65 0))
-    (property "Value" "Conn_01x02" (id 1) (at 182.88 120.65 0)
+    (property "Value" "JST SH BM02B Connector" (id 1) (at 182.88 120.65 0)
       (effects (font (size 1.27 1.27)) hide)
     )
@@
     )
     (path "/b893555e-743d-4cf9-bd5a-f020e2718f96"
-      (reference "J1") (unit 1) (value "Conn_01x02") (footprint "Connector_JST:JST_SH_BM02B-SRSS-TB_1x02-1MP_P1.00mm_Vertical")
+      (reference "J1") (unit 1) (value "JST SH BM02B Connector") (footprint "Connector_JST:JST_SH_BM02B-SRSS-TB_1x02-1MP_P1.00mm_Vertical")
     )
     (path "/41f187f0-c6dd-43c8-8895-eac8ebc41199"
-      (reference "J2") (unit 1) (value "Conn_01x02") (footprint "Connector_JST:JST_SH_BM02B-SRSS-TB_1x02-1MP_P1.00mm_Vertical")
+      (reference "J2") (unit 1) (value "JST SH BM02B Connector") (footprint "Connector_JST:JST_SH_BM02B-SRSS-TB_1x02-1MP_P1.00mm_Vertical")
     )
     (path "/1b3a272c-48df-47fd-b37c-cee5898d6c9a"
-      (reference "J3") (unit 1) (value "Conn_01x02") (footprint "Connector_JST:JST_SH_BM02B-SRSS-TB_1x02-1MP_P1.00mm_Vertical")
+      (reference "J3") (unit 1) (value "JST SH BM02B Connector") (footprint "Connector_JST:JST_SH_BM02B-SRSS-TB_1x02-1MP_P1.00mm_Vertical")
     )
     (path "/f454f6b8-6542-4029-aa53-85ac46fe0b4b"
-      (reference "J4") (unit 1) (value "Conn_01x02") (footprint "Connector_JST:JST_SH_BM02B-SRSS-TB_1x02-1MP_P1.00mm_Vertical")
+      (reference "J4") (unit 1) (value "JST SH BM02B Connector") (footprint "Connector_JST:JST_SH_BM02B-SRSS-TB_1x02-1MP_P1.00mm_Vertical")
     )
     (path "/9b7695b7-9db0-4c8e-9077-f8b7d4d3a13e"
-      (reference "J5") (unit 1) (value "Conn_01x02") (footprint "Connector_JST:JST_SH_BM02B-SRSS-TB_1x02-1MP_P1.00mm_Vertical")
+      (reference "J5") (unit 1) (value "JST SH BM02B Connector") (footprint "Connector_JST:JST_SH_BM02B-SRSS-TB_1x02-1MP_P1.00mm_Vertical")
     )
     (path "/cb8e411a-1cc5-4c53-9eeb-4024c1c299a0"
-      (reference "J6") (unit 1) (value "Conn_01x02") (footprint "Connector_JST:JST_SH_BM02B-SRSS-TB_1x02-1MP_P1.00mm_Vertical")
+      (reference "J6") (unit 1) (value "JST SH BM02B Connector") (footprint "Connector_JST:JST_SH_BM02B-SRSS-TB_1x02-1MP_P1.00mm_Vertical")
     )
     (path "/6746b76e-fcdf-48a8-9cd1-db639066bc4d"
-      (reference "J7") (unit 1) (value "Conn_01x02") (footprint "Connector_JST:JST_PH_B2B-PH-SM4-TB_1x02-1MP_P2.00mm_Vertical")
+      (reference "J7") (unit 1) (value "Conn_01x02") (footprint "Connector_JST:JST_PH_B2B-PH-K_1x02_P2.00mm_Vertical")
     )
     (path "/cc6dfe6c-2682-437b-b21c-d3c16a16c093"
@@
     )
     (path "/74652855-8612-439a-8f2e-38d2da922f50"
-      (reference "R5") (unit 1) (value "R") (footprint "Resistor_SMD:R_0805_2012Metric")
+      (reference "R5") (unit 1) (value "1.7k") (footprint "Resistor_SMD:R_0805_2012Metric")
     )
     (path "/3f231048-8615-40fd-9fc8-49df8a7de72f"
-      (reference "R6") (unit 1) (value "R") (footprint "Resistor_SMD:R_0805_2012Metric")
+      (reference "R6") (unit 1) (value "1.7k") (footprint "Resistor_SMD:R_0805_2012Metric")
     )
     (path "/d3ec3927-2308-464a-86ac-ddba9a8eef92"
